Commit message: Mon Nov 12 07:35:53 EST 2018fixed issue#8

File: ironfish_description/robots/ironfish.urdf (robot description, URDF)
Before this commit: robot rsc_car, 5 links, 4 joints
Links:
- link base_link: geometry collision mesh filename=package://ironfish_description/meshes/base_link.STL; visual mesh filename=package://ironfish_description/meshes/base_link.STL
- link hokuyo_link: geometry collision mesh filename=package://ironfish_description/meshes/hokuyo_link.STL; visual mesh filename=package://ironfish_description/meshes/hokuyo_link.STL
- link lwheel_link: geometry collision mesh filename=package://ironfish_description/meshes/lwheel_link.STL; visual mesh filename=package://ironfish_description/meshes/lwheel_link.STL
- link rwheel_link: geometry collision mesh filename=package://ironfish_description/meshes/rwheel_link.STL; visual mesh filename=package://ironfish_description/meshes/rwheel_link.STL

File: ironfish_description/robots/ironfish_materials.xacro (robot description, xacro)
@@ -1,4 +1,4 @@
 <?xml version="1.0"?>
-<robot name="rsc_car">
+<robot name="ironfish">
   <material name="black">
     <color rgba="0.0 0.0 0.0 1.0"/>

Commit message: Thu Nov 22 23:10:44 EST 2018 simulation cloud only work on empty world

File: ironfish_description/robots/ironfish.urdf (robot description, URDF)
Before this commit: robot ironfish, 5 links, 4 joints
Links:
- link base_footprint: geometry visual box size=0.1 0.1 0.1
- link hokuyo_link: mass 0 -> 1
