Commit message: Mon Dec 31 03:08:20 CST 2018 extend laser to dual-scan mode for costmap generating

File: ironfish_description/robots/ironfish.urdf.xacro (robot description, xacro)
@@ -1,7 +1,7 @@
 <?xml version="1.0"?>
 <robot name="ironfish" xmlns:xacro="http://www.ros.org/wiki/xacro">
-  <!-- Base and wheel for iubot1 -->
+  <!-- Base and wheel for ironfish -->
   <xacro:include filename="$(find ironfish_description)/urdf/base/base.urdf.xacro"/>
-  <!-- colors for iubot1 -->
+  <!-- colors for ironfish -->
   <xacro:include filename="$(find ironfish_description)/urdf/materials.xacro"/>
   <!-- Gazebo plugin -->

File: ironfish_description/urdf/base/base.urdf.xacro (robot description, xacro)
@@ -171,4 +171,5 @@
     <!-- Hokuyo utm30lx-->
     <xacro:hokuyo_utm30lx name="hokuyo" parent="base_link"/>
+    <xacro:hokuyo_utm30lx_back name="hokuyo_back" parent="base_link"/>
     <!-- Extensions -->
     <xacro:ironfish_base_gazebo/>

File: ironfish_description/urdf/sensors/hokuyo_utm30lx.urdf.xacro (robot description, xacro)
@@ -5,5 +5,5 @@
     <joint name="${name}_joint" type="fixed">
       <!--origin xyz="0.105 0.000 0.229" rpy="0 0 0" /-->
-      <origin xyz="0.105 0.006 0.229" rpy="0 0 0" />
+      <origin xyz="0.130 0.006 0.229" rpy="0 0 0" />
       <parent link="${parent}"/>
       <child link="${name}_link"/>
@@ -31,3 +31,32 @@
     <xacro:hokuyo_utm30lx_gazebo name="${name}" ros_topic="/scan" update_rate="40" ray_count="720" min_angle="-2" max_angle="2"/>
   </xacro:macro>
+  <xacro:macro name="hokuyo_utm30lx_back" params="name parent">
+    <joint name="${name}_joint" type="fixed">
+      <!--origin xyz="0.105 0.000 0.229" rpy="0 0 0" /-->
+      <origin xyz="-0.180 0.006 0.229" rpy="0 0 3.1415926535897931" />
+      <parent link="${parent}"/>
+      <child link="${name}_link"/>
+    </joint>
+    <link name="${name}_link">
+      <!--inertial>
+        <mass value="0.0000000270" />
+        <origin xyz="0 0 0" rpy="0 0 0" />
+        <inertia ixx="2.632e-4" ixy="0" ixz="0" iyy="2.632e-4" iyz="0" izz="2.632e-4" />
+      </inertial-->
+      <visual>
+        <origin xyz="0 0 0" rpy="0 0 0" />
+        <geometry>
+        <mesh filename="package://ironfish_description/meshes/hokuyo_utm30lx/hokuyo_utm_30lx.dae"/>
+      </geometry>
+      </visual>
+      <collision>
+        <origin xyz="0 0 0" rpy="0 0 0" />
+        <geometry>
+        <box size="0.058 0.058 0.087" />
+      </geometry>
+      </collision>
+    </link>
+    <!-- extensions -->
+    <xacro:hokuyo_utm30lx_gazebo name="${name}" ros_topic="/scan2" update_rate="40" ray_count="720" min_angle="-2" max_angle="2"/>
+  </xacro:macro>
 </robot>

Commit message: Tue Jun 11 21:20:30 CST 2019 debug of imu on ironfish, now work fine with cartographer

File: ironfish_description/robots/ironfish.urdf.xacro (robot description, xacro)
@@ -27,7 +27,7 @@
     <plugin name="imu_controller" filename="libhector_gazebo_ros_imu.so">
       <robotNamespace>/</robotNamespace>
-      <frameId>base_link</frameId>
+      <frameId>imu_base_link</frameId>
       <updateRate>50.0</updateRate>
-      <bodyName>base_link</bodyName>
+      <bodyName>imu_base_link</bodyName>
       <topicName>imu/data</topicName>
       <accelDrift>0.005 0.005 0.005</accelDrift>

File: ironfish_description/urdf/base/base.urdf.xacro (robot description, xacro)
@@ -167,4 +167,30 @@
         </collision>
       </link>
+    <!-- Sparkfun imu-->
+    <joint name="imu_joint" type="fixed">
+      <axis xyz="0 0 0"/> <!-- 0 1 0 -->
+      <origin xyz="0 0 0"/>
+      <parent link="base_link"/>
+      <child link="base_imu_link"/>
+    </joint>
+    <link name="base_imu_link">
+      <inertial>
+        <mass value="0.001"/>
+        <origin rpy="0 0 0" xyz="0 0 0"/>
+        <inertia ixx="0.0001" ixy="0" ixz="0" iyy="0.000001" iyz="0" izz="0.0001"/>
+      </inertial>
+      <visual>
+        <origin rpy="0 0 0" xyz="0 0 0"/>
+        <geometry>
+          <box size="0.001 0.001 0.001"/>
+        </geometry>
+      </visual>
+      <collision>
+        <origin rpy="0 0 0" xyz="0 0 0"/>
+        <geometry>
+          <box size=".001 .001 .001"/>
+        </geometry>
+      </collision>
+    </link>
     <!-- Intel realsense-->
     <sensor_d435 parent="base_link">
