Commit message: Fri Nov 30 07:39:13 EST 2018 fixed the migration bugs

File: ironfish_description/urdf/sensors/hokuyo_utm30lx.urdf.xacro (robot description, xacro)
@@ -1,5 +1,5 @@
 <?xml version="1.0"?>
 <robot xmlns:xacro="http://ros.org/wiki/xacro">
-  <xacro:include filename="$(find rsc_car_description)/urdf/sensors/hokuyo_utm30lx.gazebo.xacro" />
+  <xacro:include filename="$(find ironfish_description)/urdf/sensors/hokuyo_utm30lx.gazebo.xacro" />
   <xacro:macro name="hokuyo_utm30lx" params="name parent">
     <joint name="${name}_joint" type="fixed">
@@ -18,5 +18,5 @@
         <origin xyz="0 0 0" rpy="0 0 0" />
         <geometry>
-        <mesh filename="package://rsc_car_description/meshes/hokuyo_utm30lx/hokuyo_utm_30lx.dae"/>
+        <mesh filename="package://ironfish_description/meshes/hokuyo_utm30lx/hokuyo_utm_30lx.dae"/>
       </geometry>
       </visual>
