Commit message: Tue Dec  4 09:50:16 EST 2018 fixed the random dift problem cause by the reponse ok from controller

File: ironfish_description/urdf/base/base.gazebo.xacro (robot description, xacro)
@@ -13,5 +13,5 @@
   </xacro:macro>
   <!-- Right and left wheels -->
-  <xacro:macro name="ironfish_rl_wheel_gazebo">
+  <xacro:macro name="ironfish_rwheel_gazebo">
     <gazebo reference="right_wheel">
       <material>Gazebo/Black</material>
@@ -23,4 +23,6 @@
       <dampingFactor value="0.1"/>
     </gazebo>
+  </xacro:macro>
+  <xacro:macro name="ironfish_lwheel_gazebo">
     <gazebo reference="left_wheel">
       <material>Gazebo/Black</material>

File: ironfish_description/urdf/base/base.urdf.xacro (robot description, xacro)
@@ -5,5 +5,5 @@
   <xacro:include filename="$(find ironfish_description)/urdf/sensors/hokuyo_utm30lx.urdf.xacro" />
   <xacro:property name="pi" value="3.1415926535897931" />
-  <xacro:macro name="r_wheel">
+  <xacro:macro name="rwheel">
     <link name="rwheel_link">
       <inertial>
@@ -57,8 +57,8 @@
     </joint>
     <!-- Extensions -->
-    <xacro:ironfish_rl_wheel_gazebo/>
+    <xacro:ironfish_rwheel_gazebo/>
     <xacro:ironfish_rwheel_trans/>
   </xacro:macro>
-  <xacro:macro name="l_wheel">
+  <xacro:macro name="lwheel">
     <link name="lwheel_link">
       <inertial>
@@ -112,5 +112,5 @@
     </joint>
     <!-- Extensions -->
-    <xacro:ironfish_rl_wheel_gazebo/>
+    <xacro:ironfish_lwheel_gazebo/>
     <xacro:ironfish_lwheel_trans/>
   </xacro:macro>
@@ -167,6 +167,6 @@
       </link>
     <!-- Wheel macros -->
-    <xacro:r_wheel />
-    <xacro:l_wheel />
+    <xacro:rwheel />
+    <xacro:lwheel />
     <!-- Hokuyo utm30lx-->
     <xacro:hokuyo_utm30lx name="hokuyo" parent="base_link"/>
