Commit message: Thu Feb 28 01:25:21 CST 2019 added realsense gazebo model, modified laser height, modified footprint height.

File: ironfish_description/urdf/base/base.urdf.xacro (robot description, xacro)
@@ -4,4 +4,5 @@
   <xacro:include filename="$(find ironfish_description)/urdf/base/base.gazebo.xacro" />
   <xacro:include filename="$(find ironfish_description)/urdf/sensors/hokuyo_utm30lx.urdf.xacro" />
+  <xacro:include filename="$(find ironfish_description)/urdf/sensors/_d435.urdf.xacro" />
   <xacro:property name="pi" value="3.1415926535897931" />
   <xacro:macro name="rwheel">
@@ -30,5 +31,5 @@
         </geometry>
         <material
-          name="black">
+          name="white">
         </material>
       </visual>
@@ -85,5 +86,5 @@
         </geometry>
         <material
-          name="black">
+          name="white">
         </material>
       </visual>
@@ -115,5 +116,5 @@
     <xacro:ironfish_lwheel_trans/>
   </xacro:macro>
-    <xacro:macro name="ironfish_base">
+  <xacro:macro name="ironfish_base">
       <link name="base_footprint">
         <visual>
@@ -125,5 +126,5 @@
       </link>
       <joint name="base_footprint_joint" type="fixed">
-        <origin xyz="0 0 0.1124430740677247" rpy="0 0 0" />
+        <origin xyz="0 0 0.1014430740677247" rpy="0 0 0" />
         <child link="base_link" />
         <parent link="base_footprint"/>
@@ -166,4 +167,8 @@
         </collision>
       </link>
+    <!-- Intel realsense-->
+    <sensor_d435 parent="base_link">
+      <origin xyz="0.130 0.006 0.229" rpy="0 0 0"/>
+    </sensor_d435>
     <!-- Wheel macros -->
     <xacro:rwheel />

File: ironfish_description/urdf/sensors/hokuyo_utm30lx.urdf.xacro (robot description, xacro)
@@ -5,5 +5,5 @@
     <joint name="${name}_joint" type="fixed">
       <!--origin xyz="0.105 0.000 0.229" rpy="0 0 0" /-->
-      <origin xyz="0.130 0.006 0.229" rpy="0 0 0" />
+      <origin xyz="0.130 0.006 0.0914430740677247" rpy="0 0 0" />
       <parent link="${parent}"/>
       <child link="${name}_link"/>
@@ -34,5 +34,5 @@
     <joint name="${name}_joint" type="fixed">
       <!--origin xyz="0.105 0.000 0.229" rpy="0 0 0" /-->
-      <origin xyz="-0.180 0.006 0.229" rpy="0 0 3.1415926535897931" />
+      <origin xyz="-0.180 0.006 0.0914430740677247" rpy="0 0 3.1415926535897931" />
       <parent link="${parent}"/>
       <child link="${name}_link"/>

Commit message: Mon Jun 10 21:23:01 CST 2019 add calibrated realsense height and precise location

File: ironfish_description/urdf/base/base.urdf.xacro (robot description, xacro)
@@ -169,5 +169,6 @@
     <!-- Intel realsense-->
     <sensor_d435 parent="base_link">
-      <origin xyz="0.130 0.006 0.229" rpy="0 0 0"/>
+      <!--origin xyz="0.135 0.006 0.178" rpy="0 0 0"/--> <!-- align the front edge-->
+      <origin xyz="0.047 0.006 0.463" rpy="0 0 0"/> <!--real measure from blue extend version-->
     </sensor_d435>
     <!-- Wheel macros -->

Commit message: Thu Jun 13 22:37:10 CST 2019 give the true location of imu, but it seems still not work better

File: ironfish_description/urdf/base/base.urdf.xacro (robot description, xacro)
@@ -170,5 +170,5 @@
     <joint name="imu_joint" type="fixed">
       <axis xyz="0 0 0"/> <!-- 0 1 0 -->
-      <origin xyz="0 0 0"/>
+      <origin xyz="0.0455 0.006 0.464"/>
       <parent link="base_link"/>
       <child link="base_imu_link"/>
